File: gauge_servo.kicad_sch (KiCad schematic)
At the start: 32 parts, among them J1 Servo 1, J10 LIM1, J11 LIM2, J12 NPX1, J3 Servo 2, J4 I2C, J5 STEPPER, J6 INPUT_1, J7 NPX2, J8 INPUT_2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

Commit message: Fixed pinout error or Adafruit TB6612 custom component that caused short between 5V and gnd
Connections:
- net +5V: now also U3.18 (VMOTOR+); no longer U3.17 (VMOTOR+)
- net GND: now also U3.17 (VMOTOR-); no longer U3.18 (VMOTOR-)
Changed lines of the file:
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@@
     )
   )
-  (symbol (lib_id "power:GND") (at 237.49 29.21 0) (unit 1)
+  (symbol (lib_name "GND_5") (lib_id "power:GND") (at 237.49 29.21 0) (unit 1)
     (in_bom yes) (on_board yes) (fields_autoplaced)
     (property "Reference" "#PWR08" (id 0) (at 237.49 35.56 0)
@@
     (pin "1")
   )
-  (symbol (lib_id "power:+5V") (at 189.23 20.32 0) (unit 1)
+  (symbol (lib_name "+5V_2") (lib_id "power:+5V") (at 189.23 20.32 0) (unit 1)
     (in_bom yes) (on_board yes) (fields_autoplaced)
     (property "Reference" "#PWR01" (id 0) (at 189.23 24.13 0)
@@
     (pin "1")
   )
-  (symbol (lib_id "power:+3V3") (at 115.57 40.64 0) (unit 1)
+  (symbol (lib_name "+3V3_1") (lib_id "power:+3V3") (at 115.57 40.64 0) (unit 1)
     (in_bom yes) (on_board yes) (fields_autoplaced)
     (property "Reference" "#PWR05" (id 0) (at 115.57 44.45 0)
@@
     (pin "4")
   )
-  (symbol (lib_id "power:+12V") (at 49.53 157.48 0) (unit 1)
+  (symbol (lib_name "+12V_3") (lib_id "power:+12V") (at 49.53 157.48 0) (unit 1)
     (in_bom yes) (on_board yes) (fields_autoplaced)
     (property "Reference" "#PWR023" (id 0) (at 49.53 161.29 0)
@@
     (pin "9")
   )
-  (symbol (lib_id "power:+5V") (at 237.49 21.59 0) (unit 1)
+  (symbol (lib_name "+5V_5") (lib_id "power:+5V") (at 237.49 21.59 0) (unit 1)
     (in_bom yes) (on_board yes) (fields_autoplaced)
     (property "Reference" "#PWR07" (id 0) (at 237.49 25.4 0)
@@
     (pin "1")
   )
-  (symbol (lib_id "power:+5V") (at 251.46 139.7 0) (unit 1)
+  (symbol (lib_name "+5V_9") (lib_id "power:+5V") (at 251.46 139.7 0) (unit 1)
     (in_bom yes) (on_board yes) (fields_autoplaced)
     (property "Reference" "#PWR022" (id 0) (at 251.46 143.51 0)
@@
     (pin "1")
   )
-  (symbol (lib_id "power:GND") (at 248.92 58.42 0) (unit 1)
+  (symbol (lib_name "GND_4") (lib_id "power:GND") (at 248.92 58.42 0) (unit 1)
     (in_bom yes) (on_board yes) (fields_autoplaced)
     (property "Reference" "#PWR015" (id 0) (at 248.92 64.77 0)
@@
     (pin "1")
   )
-  (symbol (lib_id "power:GND") (at 214.63 100.33 0) (unit 1)
+  (symbol (lib_name "GND_10") (lib_id "power:GND") (at 214.63 100.33 0) (unit 1)
     (in_bom yes) (on_board yes) (fields_autoplaced)
     (property "Reference" "#PWR019" (id 0) (at 214.63 106.68 0)
@@
     (pin "1")
   )
-  (symbol (lib_id "power:GND") (at 43.18 82.55 0) (unit 1)
+  (symbol (lib_name "GND_2") (lib_id "power:GND") (at 43.18 82.55 0) (unit 1)
     (in_bom yes) (on_board yes) (fields_autoplaced)
     (property "Reference" "#PWR014" (id 0) (at 43.18 88.9 0)
@@
     (pin "2")
   )
-  (symbol (lib_id "power:GND") (at 148.59 149.86 0) (unit 1)
+  (symbol (lib_name "GND_6") (lib_id "power:GND") (at 148.59 149.86 0) (unit 1)
     (in_bom yes) (on_board yes) (fields_autoplaced)
     (property "Reference" "#PWR038" (id 0) (at 148.59 156.21 0)
@@
     (pin "3")
   )
-  (symbol (lib_id "power:+5V") (at 218.44 53.34 0) (unit 1)
+  (symbol (lib_name "+5V_6") (lib_id "power:+5V") (at 218.44 53.34 0) (unit 1)
     (in_bom yes) (on_board yes) (fields_autoplaced)
     (property "Reference" "#PWR011" (id 0) (at 218.44 57.15 0)
@@
     (pin "2")
   )
-  (symbol (lib_id "power:GND") (at 189.23 27.94 0) (unit 1)
+  (symbol (lib_name "GND_3") (lib_id "power:GND") (at 189.23 27.94 0) (unit 1)
     (in_bom yes) (on_board yes) (fields_autoplaced)
     (property "Reference" "#PWR02" (id 0) (at 189.23 34.29 0)
@@
     (pin "1")
   )
-  (symbol (lib_id "power:GND") (at 43.18 180.34 0) (unit 1)
+  (symbol (lib_name "GND_8") (lib_id "power:GND") (at 43.18 180.34 0) (unit 1)
     (in_bom yes) (on_board yes) (fields_autoplaced)
     (property "Reference" "#PWR028" (id 0) (at 43.18 186.69 0)
@@
     (pin "1")
   )
-  (symbol (lib_id "power:+5V") (at 148.59 166.37 0) (unit 1)
+  (symbol (lib_name "+5V_7") (lib_id "power:+5V") (at 148.59 166.37 0) (unit 1)
     (in_bom yes) (on_board yes) (fields_autoplaced)
     (property "Reference" "#PWR039" (id 0) (at 148.59 170.18 0)
@@
     (pin "2")
   )
-  (symbol (lib_id "power:GND") (at 43.18 134.62 0) (unit 1)
+  (symbol (lib_name "GND_12") (lib_id "power:GND") (at 43.18 134.62 0) (unit 1)
     (in_bom yes) (on_board yes) (fields_autoplaced)
     (property "Reference" "#PWR021" (id 0) (at 43.18 140.97 0)
@@
     (pin "1")
   )
-  (symbol (lib_id "power:GND") (at 76.2 48.26 0) (unit 1)
+  (symbol (lib_name "GND_1") (lib_id "power:GND") (at 76.2 48.26 0) (unit 1)
     (in_bom yes) (on_board yes)
     (property "Reference" "#PWR06" (id 0) (at 76.2 54.61 0)
@@
     (pin "1")
   )
-  (symbol (lib_id "power:GND") (at 35.56 125.73 0) (unit 1)
+  (symbol (lib_name "GND_11") (lib_id "power:GND") (at 35.56 125.73 0) (unit 1)
     (in_bom yes) (on_board yes) (fields_autoplaced)
     (property "Reference" "#PWR020" (id 0) (at 35.56 132.08 0)
@@
     (pin "3")
   )
-  (symbol (lib_id "power:+12V") (at 35.56 162.56 0) (unit 1)
+  (symbol (lib_name "+12V_4") (lib_id "power:+12V") (at 35.56 162.56 0) (unit 1)
     (in_bom yes) (on_board yes) (fields_autoplaced)
     (property "Reference" "#PWR026" (id 0) (at 35.56 166.37 0)
@@
     (pin "1")
   )
-  (symbol (lib_id "power:+5V") (at 76.2 40.64 0) (unit 1)
+  (symbol (lib_name "+5V_1") (lib_id "power:+5V") (at 76.2 40.64 0) (unit 1)
     (in_bom yes) (on_board yes) (fields_autoplaced)
     (property "Reference" "#PWR04" (id 0) (at 76.2 44.45 0)
@@
     (pin "1")
   )
-  (symbol (lib_id "power:+5V") (at 184.15 55.88 0) (unit 1)
+  (symbol (lib_name "+5V_4") (lib_id "power:+5V") (at 184.15 55.88 0) (unit 1)
     (in_bom yes) (on_board yes) (fields_autoplaced)
     (property "Reference" "#PWR013" (id 0) (at 184.15 59.69 0)
@@
     (pin "1")
   )
-  (symbol (lib_id "power:GND") (at 35.56 171.45 0) (unit 1)
+  (symbol (lib_name "GND_9") (lib_id "power:GND") (at 35.56 171.45 0) (unit 1)
     (in_bom yes) (on_board yes) (fields_autoplaced)
     (property "Reference" "#PWR027" (id 0) (at 35.56 177.8 0)
@@
     (pin "1")
   )
-  (symbol (lib_id "power:+3V3") (at 43.18 80.01 0) (unit 1)
+  (symbol (lib_name "+3V3_2") (lib_id "power:+3V3") (at 43.18 80.01 0) (unit 1)
     (in_bom yes) (on_board yes) (fields_autoplaced)
     (property "Reference" "#PWR012" (id 0) (at 43.18 83.82 0)
@@
     (pin "1")
   )
-  (symbol (lib_id "power:+3V3") (at 213.36 53.34 0) (unit 1)
+  (symbol (lib_name "+3V3_3") (lib_id "power:+3V3") (at 213.36 53.34 0) (unit 1)
     (in_bom yes) (on_board yes) (fields_autoplaced)
     (property "Reference" "#PWR010" (id 0) (at 213.36 57.15 0)
@@
     (pin "2")
   )
-  (symbol (lib_id "power:+3V3") (at 69.85 157.48 0) (unit 1)
+  (symbol (lib_name "+3V3_4") (lib_id "power:+3V3") (at 69.85 157.48 0) (unit 1)
     (in_bom yes) (on_board yes) (fields_autoplaced)
     (property "Reference" "#PWR024" (id 0) (at 69.85 161.29 0)
@@
     (pin "2")
   )
-  (symbol (lib_id "power:+5V") (at 148.59 129.54 0) (unit 1)
+  (symbol (lib_name "+5V_8") (lib_id "power:+5V") (at 148.59 129.54 0) (unit 1)
     (in_bom yes) (on_board yes) (fields_autoplaced)
     (property "Reference" "#PWR034" (id 0) (at 148.59 133.35 0)
@@
     (pin "1")
   )
-  (symbol (lib_id "power:GND") (at 251.46 125.73 0) (unit 1)
+  (symbol (lib_name "GND_13") (lib_id "power:GND") (at 251.46 125.73 0) (unit 1)
     (in_bom yes) (on_board yes) (fields_autoplaced)
     (property "Reference" "#PWR042" (id 0) (at 251.46 132.08 0)
@@
     (pin "1")
   )
-  (symbol (lib_id "power:GND") (at 148.59 186.69 0) (unit 1)
+  (symbol (lib_name "GND_7") (lib_id "power:GND") (at 148.59 186.69 0) (unit 1)
     (in_bom yes) (on_board yes) (fields_autoplaced)
     (property "Reference" "#PWR040" (id 0) (at 148.59 193.04 0)
@@
     (pin "4")
   )
-  (symbol (lib_id "power:+5V") (at 248.92 50.8 0) (unit 1)
+  (symbol (lib_name "+5V_3") (lib_id "power:+5V") (at 248.92 50.8 0) (unit 1)
     (in_bom yes) (on_board yes) (fields_autoplaced)
     (property "Reference" "#PWR09" (id 0) (at 248.92 54.61 0)
@@
     (pin "3")
   )
-  (symbol (lib_id "power:+12V") (at 35.56 116.84 0) (unit 1)
+  (symbol (lib_name "+12V_2") (lib_id "power:+12V") (at 35.56 116.84 0) (unit 1)
     (in_bom yes) (on_board yes) (fields_autoplaced)
     (property "Reference" "#PWR018" (id 0) (at 35.56 120.65 0)
@@
     (pin "3")
   )
-  (symbol (lib_id "power:+12V") (at 46.99 40.64 0) (unit 1)
+  (symbol (lib_name "+12V_1") (lib_id "power:+12V") (at 46.99 40.64 0) (unit 1)
     (in_bom yes) (on_board yes) (fields_autoplaced)
     (property "Reference" "#PWR03" (id 0) (at 46.99 44.45 0)
